File: 2611332-Ana Irizar-MicroDuino/2611332-Ana Irizar-MicroDuino.kicad_pcb (KiCad board)
At the start: 2 copper layers, 14 parts, among them J1 Conn_01x10_Socket, J2 USB_A, U1 ATtiny85-20S

Commit message: actualizo mi pcb
Parts:
- moved D2 86.9 mm to (77.6, 124.5)
- moved D5 81.7 mm to (79.6, 132.5)
- moved R3 76.5 mm to (86.7, 135.6)
- moved R1 74.6 mm to (87.3, 127.4), turned to 90 degrees
- moved D4 71.4 mm to (99.8, 129.0)
- moved R4 68.1 mm to (81.0, 135.5), turned to 90 degrees
- moved R2 64.3 mm to (100.2, 125.0)
- moved C1 63.5 mm to (79.3, 128.8), turned to -90 degrees
- moved U1 59.0 mm to (93.7, 133.3)
- moved J2 56.2 mm to (78.5, 118.1)
- moved D1 56.1 mm to (74.4, 131.6)
- moved R5 55.9 mm to (82.7, 125.8)
- moved J1 55.6 mm to (77.0, 139.2)
- moved D3 50.8 mm to (93.4, 124.4)
Routing:
- net GND: track 0.97 -> 98.9 mm, vias 0 -> 7
- net +5V: track 1.57 -> 54.4 mm, vias 2 -> 0
- net Net-(D1-K): track 5.67 -> 45.9 mm, vias 2 -> 6
- net Net-(J1-Pin_8): track 0.00 -> 38.5 mm
- net Net-(D4-A): track 0.00 -> 28.9 mm
- net Net-(D3-A): track 0.00 -> 24.5 mm
- net Net-(J1-Pin_7): track 0.00 -> 17.7 mm, vias 0 -> 2
- net Net-(J1-Pin_4): track 0.00 -> 12.1 mm
- net Net-(D5-K): track 0.00 -> 9.92 mm
- net Net-(J1-Pin_6): track 0.00 -> 5.59 mm, vias 0 -> 1
- net Net-(D4-K): track 0.00 -> 4.02 mm, vias 0 -> 3
- net Net-(J1-Pin_9): track 0.00 -> 3.94 mm, vias 0 -> 1
Other:
- board outline added: 30.6 x 28.5 mm
